File: tester_board.kicad_pcb (KiCad board)
At the start: 2 copper layers, 27 parts, among them J1 Conn_01x06_Male, J10 Conn_01x06_Male, J11 Conn_01x06_Male, J2 Conn_01x02, J3 USB_OTG, J4 Conn_01x06_Male, J5 Conn_01x06_Male, J6 Conn_01x06_Male, J7 USB_OTG, J8 Conn_01x02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

Commit message: finished
Parts:
- added J12: Conn_01x05, Socket_Strips:Socket_Strip_Straight_1x05_Pitch2.54mm, F.Cu at (46.7, 116.3)
- added R7: 0, Resistors_SMD:R_0603, F.Cu at (43.6, 131.7)
- added R8: 4.7k, Resistors_SMD:R_0603, F.Cu at (54.8, 82.0)
- added REF**: MountingHole_3.2mm_M3, Mounting_Holes:MountingHole_3.2mm_M3, F.Cu at (111.5, 110.5)
- added REF**: MountingHole_3.2mm_M3, Mounting_Holes:MountingHole_3.2mm_M3, F.Cu at (58.2, 115.3)
- added REF**: MountingHole_3.2mm_M3, Mounting_Holes:MountingHole_3.2mm_M3, F.Cu at (112.1, 75.6)
- J4: value Conn_01x06_Male -> Conn_01x10_Female; footprint Pin_Headers:Pin_Header_Straight_1x06_Pitch2.54mm -> Socket_Strips:Socket_Strip_Straight_1x10_Pitch2.54mm
- moved J4 12.6 mm to (40.2, 108.8)
- moved J7 4.32 mm to (38.4, 101.1)
Connections:
- J4 pad 1: Net-(J4-Pad1) -> GND
- J4 pad 2: Net-(J4-Pad2) -> /CTS
- J4 pad 3: Net-(J4-Pad3) -> /TX
- J4 pad 4: Net-(J4-Pad4) -> /RTS
- J4 pad 5: Net-(J4-Pad5) -> /RX
- J4 pad 6: Net-(J4-Pad6) -> /CBUS2
Routing:
- net /RX: track 0.00 -> 48.9 mm
- net /TX: track 0.00 -> 38.1 mm
- net /CTS: track 0.00 -> 8.60 mm
- net VCC: track 210.2 -> 218.6 mm
- net /RTS: track 0.00 -> 7.55 mm
- net /CBUS0: track 0.00 -> 6.60 mm
- net /CBUS2: track 0.00 -> 6.60 mm
- net /CBUS1: track 0.00 -> 6.60 mm
- net Net-(J7-Pad1): track 36.3 -> 32.0 mm
- net /D-: track 28.1 -> 25.4 mm
- net /D+: track 28.8 -> 26.1 mm
- net Net-(J4-Pad10): track 0.00 -> 2.64 mm
- net /MCLR: track 17.2 -> 18.1 mm
Other:
- board outline added: 85 x 69.8 mm
- board text added: "BAT_MEAS"
- board text added: "CBUS1"
- board text added: "CBUS2 CBUS0"
- board text added: "CTS"
- board text added: "MCLR VCC GND PGD PGC"
- board text added: "PWR_MEAS"
- board text added: "RA2 RA3 RA4 RA5 RA7 RA6"
- board text added: "RB4 RB3 RB2 RC0 RC1 RC2"
- board text added: "RTS"
